File: klxecu.kicad_sch (KiCad schematic)
At the start: 64 parts

Commit message: Schematic mostly complete, missing control for subthrottle valve
Parts:
- added C? (x2): u1, Capacitors_THT:C_Disc_D3.8mm_W2.6mm_P2.50mm, symbol Device:C
- added C?: 10u, Capacitors_THT:CP_Radial_Tantal_D6.0mm_P2.50mm, symbol Device:CP
- added C? (x4): 100n, symbol Device:C_Small
- added C?: 47u, Capacitors_THT:CP_Radial_Tantal_D6.0mm_P2.50mm, symbol Device:CP
- added C?: 22pf, symbol Device:C_Small
- added C?: 0.1u, symbol Device:C_Small
- added D?: 1N5818, Diode_THT:D_DO-41_SOD81_P7.62mm_Horizontal, symbol Device:D_Schottky
- added D?: 1N5919BG, Diode_THT:D_DO-41_SOD81_P7.62mm_Horizontal, symbol Device:D_Zener
- added J?: Arduino Comms Header, symbol Connector:Conn_01x06_Male
- added J?: ICSP, symbol Connector_Generic:Conn_02x03_Odd_Even
- added JP?: O2 HEAT ENABLE, symbol Jumper:Jumper_3_Open
- added R? (x3): 10k, symbol Device:R_Small
- added R?: 1M, symbol Device:R_Small
- added R?: 27, symbol Device:R_Small
- added U? (x4): 74LS14, Package_DIP:DIP-14_W7.62mm, symbol 74xx:74LS14
- added U?: LM2940T-5.0, TO_SOT_Packages_THT:TO-220_Vertical, symbol NO2C-rescue:7805-RESCUE-KARTDUINO_V0.1.1
- added U?: ATmega2560-16A, Package_QFP:TQFP-100_14x14mm_P0.5mm, symbol MCU_Microchip_ATmega:ATmega2560-16A
- added U? (x4): 74LS02, symbol 74xx:74LS02
- added U?: ERZ, Varistors:RV_Disc_D15.5_W4.2_P7.5, symbol Device:Varistor
- added Y?: 16 mhz, symbol Device:Crystal_GND3_Small
Connections:
- net KDS DIAG is gone; now on net +5V: J?.10 (Pin_10)
- net +12V: now also C?.1, C?.1, D?.2 (A), JP?.3 (B), U?.1
- net +5V: now also C?.1, C?.1, C?.1, C?.1, C?.1, C?.2, C?.2, C?.2, C?.2, C?.2, D?.1 (K), J?.1 (Pin_1), J?.2 (Pin_2), J?.2 (Pin_2), J?.3 (Pin_3), J?.6 (Pin_6), JP?.1 (A), R?.1, R?.1, R?.1, U?.10 (VCC), U?.100 (AVCC), U?.11 (GND), U?.14 (VCC), U?.14 (VCC), U?.3 (VO), U?.31 (VCC), U?.32 (GND), U?.61 (VCC), U?.62 (GND), U?.7 (GND), U?.7 (GND), U?.80 (VCC), U?.81 (GND), U?.99 (GND), Y?.3
- net ARDUINO-A0: now also U?.97 (PF0)
- net ARDUINO-A1: now also U?.96 (PF1)
- net ARDUINO-A2: now also U?.95 (PF2)
- net ARDUINO-A3: now also U?.94 (PF3)
- net ARDUINO-A4: now also U?.93 (PF4)
- net ARDUINO-A5: now also U?.92 (PF5)
- net ARDUINO-D19: now also U?.45 (PD2)
- net ARDUINO-D23: now also U?.77 (PA1)
- net ARDUINO-D4: now also U?.1 (PG5)
- net ARDUINO-D5: now also U?.5 (PE3)
- net ARDUINO-D6: now also U?.15 (PH3)
- net ARDUINO-D7: now also U?.16 (PH4)
- net ARDUINO-D8: now also U?.17 (PH5)
- net Earth: now also C?.2, C?.2, C?.2, C?.2, D?.2 (A), U?.2, U?.2 (GND)
- net KICKSTAND SW: now also R?.2, U?.5
- net NEUTRAL SW: now also R?.2, U?.3
- net O2S HEAT +: now also JP?.2 (C)
- net Vehicle Down: now also U?.1
- net SELF DIAG renamed ARDUINO-D3
- net ARDUINO-D3: now also R?.2, U?.7 (PE5)
- new net: D?.1 (K), U?.1 (VI)
- new net: U?.6, U?.6
- new net: J?.4 (Pin_4), U?.2 (PE0)
- new net: J?.5 (Pin_5), U?.3 (PE1)
- new net: C?.1, J?.6 (Pin_6)
- new net: J?.3 (Pin_3), U?.20 (PB1)
- new net: J?.4 (Pin_4), U?.21 (PB2)
- new net: J?.1 (Pin_1), U?.22 (PB3)
- new net: R?.1, U?.33 (XTAL2), Y?.2
- new net: R?.2, U?.34 (XTAL1)
- new net: C?.1, U?.98 (AREF)
- new net: R?.1, R?.2, Y?.1
- new net: U?.2, U?.2
- new net: U?.11, U?.12, U?.4
- new net: U?.4, U?.5
- new net: U?.13, U?.3
- new net ARDUINO-RST: C?.1, C?.2, J?.5 (Pin_5), U?.1, U?.30 (~{RESET})
Other:
- note added: "Kawasaki Diag (Unsupported)"
- note added: "Power Supply"
- note added: "Safety Switches"
- note added: "Self Diagnosis"
- moved on the sheet: IC?

Commit message: All sensors and components (minus subthrottle actuator)
Parts:
- added D4, D5: 1N4004, Diode_THT:D_DO-41_SOD81_P10.16mm_Horizontal, symbol Diode:1N4004
- added unit 3 of U4
- gave numbers to parts that had none: 87
- renumbered LED2 to LED4
Connections:
- net ARDUINO-D6: now also D5.2 (A); no longer R26.1, R27.2
- net ARDUINO-RST: now also U4.8, U4.9
- new net: D4.1 (K), D5.1 (K), R26.1, R27.2
- new net: D4.2 (A), U4.10
Other:
- moved on the sheet: C23, C24, C25, C26, D1, D6, R24, R25, R26, R27, U3, U4A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

Commit message: Add jumper to RST -> CHECK ENGINE output
Parts:
- added JP?: SolderJumper_2_Open, symbol Jumper:SolderJumper_2_Open
Connections:
- net at D5.1 (K), R26.1, R27.2: now also JP?.2 (B); no longer D4.1 (K)
- new net: D4.1 (K), JP?.1 (A)
Other:
- moved on the sheet: D4, U4C
Changed lines of the file:
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@@
   (junction (at 55.88 73.66) (diameter 0) (color 0 0 0 0)
   )
-  (junction (at 285.75 144.78) (diameter 0) (color 0 0 0 0)
+  (junction (at 298.45 153.67) (diameter 0) (color 0 0 0 0)
   )
   (junction (at 295.91 86.36) (diameter 0) (color 0 0 0 0)
@@
     (stroke (width 0) (type default) (color 0 0 0 0))
   )
+  (wire (pts (xy 321.31 142.24) (xy 321.31 146.05))
+    (stroke (width 0) (type default) (color 0 0 0 0))
+  )
   (wire (pts (xy 308.61 224.79) (xy 309.88 224.79))
     (stroke (width 0) (type default) (color 0 0 0 0))
@@
     (stroke (width 0) (type default) (color 0 0 0 0))
   )
+  (wire (pts (xy 308.61 140.97) (xy 308.61 142.24))
+    (stroke (width 0) (type default) (color 0 0 0 0))
+  )
   (wire (pts (xy 331.47 116.84) (xy 331.47 121.92))
     (stroke (width 0) (type default) (color 0 0 0 0))
@@
     (stroke (width 0) (type default) (color 0 0 0 0))
   )
-  (wire (pts (xy 285.75 144.78) (xy 285.75 147.32))
+  (wire (pts (xy 298.45 153.67) (xy 298.45 156.21))
     (stroke (width 0) (type default) (color 0 0 0 0))
   )
@@
     (stroke (width 0) (type default) (color 0 0 0 0))
   )
-  (wire (pts (xy 284.48 144.78) (xy 285.75 144.78))
+  (wire (pts (xy 297.18 153.67) (xy 298.45 153.67))
     (stroke (width 0) (type default) (color 0 0 0 0))
   )
@@
     (stroke (width 0) (type default) (color 0 0 0 0))
   )
-  (wire (pts (xy 285.75 147.32) (xy 288.29 147.32))
+  (wire (pts (xy 298.45 156.21) (xy 300.99 156.21))
     (stroke (width 0) (type default) (color 0 0 0 0))
   )
@@
     (stroke (width 0) (type default) (color 0 0 0 0))
   )
-  (wire (pts (xy 303.53 144.78) (xy 308.61 144.78))
+  (wire (pts (xy 316.23 153.67) (xy 321.31 153.67))
     (stroke (width 0) (type default) (color 0 0 0 0))
   )
@@
     (stroke (width 0) (type default) (color 0 0 0 0))
   )
+  (wire (pts (xy 308.61 130.81) (xy 308.61 133.35))
+    (stroke (width 0) (type default) (color 0 0 0 0))
+  )
   (wire (pts (xy 151.13 93.98) (xy 167.64 93.98))
     (stroke (width 0) (type default) (color 0 0 0 0))
@@
     (stroke (width 0) (type default) (color 0 0 0 0))
   )
-  (wire (pts (xy 285.75 142.24) (xy 288.29 142.24))
+  (wire (pts (xy 298.45 151.13) (xy 300.99 151.13))
     (stroke (width 0) (type default) (color 0 0 0 0))
   )
@@
     (stroke (width 0) (type default) (color 0 0 0 0))
   )
-  (wire (pts (xy 308.61 137.16) (xy 308.61 130.81))
-    (stroke (width 0) (type default) (color 0 0 0 0))
-  )
   (wire (pts (xy 370.84 48.26) (xy 370.84 49.53))
     (stroke (width 0) (type default) (color 0 0 0 0))
@@
     (stroke (width 0) (type default) (color 0 0 0 0))
   )
+  (wire (pts (xy 308.61 142.24) (xy 321.31 142.24))
+    (stroke (width 0) (type default) (color 0 0 0 0))
+  )
   (wire (pts (xy 71.12 55.88) (xy 87.63 55.88))
     (stroke (width 0) (type default) (color 0 0 0 0))
@@
     (stroke (width 0) (type default) (color 0 0 0 0))
   )
-  (wire (pts (xy 285.75 144.78) (xy 285.75 142.24))
+  (wire (pts (xy 298.45 153.67) (xy 298.45 151.13))
     (stroke (width 0) (type default) (color 0 0 0 0))
   )
@@
     )
   )
-  (global_label "ARDUINO-RST" (shape output) (at 284.48 144.78 180) (fields_autoplaced)
+  (global_label "ARDUINO-RST" (shape output) (at 297.18 153.67 180) (fields_autoplaced)
     (effects (font (size 1.27 1.27)) (justify right))
-    (property "Intersheet References" "${INTERSHEET_REFS}" (id 0) (at 268.8226 144.7006 0)
+    (property "Intersheet References" "${INTERSHEET_REFS}" (id 0) (at 281.5226 153.5906 0)
       (effects (font (size 1.27 1.27)) (justify right) hide)
     )
@@
     (pin "9")
   )
+  (symbol (lib_id "Jumper:SolderJumper_2_Open") (at 308.61 137.16 90) (unit 1)
+    (in_bom yes) (on_board yes)
+    (property "Reference" "JP?" (id 0) (at 300.99 135.89 90)
+      (effects (font (size 1.27 1.27)) (justify right))
+    )
+    (property "Value" "SolderJumper_2_Open" (id 1) (at 285.75 138.43 90)
+      (effects (font (size 1.27 1.27)) (justify right))
+    )
+    (property "Footprint" "" (id 2) (at 308.61 137.16 0)
+      (effects (font (size 1.27 1.27)) hide)
+    )
+    (property "Datasheet" "~" (id 3) (at 308.61 137.16 0)
+      (effects (font (size 1.27 1.27)) hide)
+    )
+    (pin "1")
+    (pin "2")
+  )
   (symbol (lib_id "Device:R_Small") (at 372.11 127 270) (unit 1)
     (in_bom yes) (on_board yes)
@@
     (pin "2")
   )
-  (symbol (lib_id "74xx:74LS02") (at 295.91 144.78 0) (unit 3)
+  (symbol (lib_id "74xx:74LS02") (at 308.61 153.67 0) (unit 3)
     (in_bom yes) (on_board yes) (fields_autoplaced)
-    (property "Reference" "U4" (id 0) (at 295.91 135.89 0))
-    (property "Value" "74LS02" (id 1) (at 295.91 138.43 0))
-    (property "Footprint" "" (id 2) (at 295.91 144.78 0)
+    (property "Reference" "U4" (id 0) (at 308.61 144.78 0))
+    (property "Value" "74LS02" (id 1) (at 308.61 147.32 0))
+    (property "Footprint" "" (id 2) (at 308.61 153.67 0)
       (effects (font (size 1.27 1.27)) hide)
     )
-    (property "Datasheet" "http://www.ti.com/lit/gpn/sn74ls02" (id 3) (at 295.91 144.78 0)
+    (property "Datasheet" "http://www.ti.com/lit/gpn/sn74ls02" (id 3) (at 308.61 153.67 0)
       (effects (font (size 1.27 1.27)) hide)
     )
@@
     (pin "2")
   )
-  (symbol (lib_id "Diode:1N4004") (at 308.61 140.97 90) (mirror x) (unit 1)
+  (symbol (lib_id "Diode:1N4004") (at 321.31 149.86 90) (mirror x) (unit 1)
     (in_bom yes) (on_board yes) (fields_autoplaced)
-    (property "Reference" "D4" (id 0) (at 311.15 139.6999 90)
+    (property "Reference" "D4" (id 0) (at 323.85 148.5899 90)
       (effects (font (size 1.27 1.27)) (justify right))
     )
-    (property "Value" "1N4004" (id 1) (at 311.15 142.2399 90)
+    (property "Value" "1N4004" (id 1) (at 323.85 151.1299 90)
       (effects (font (size 1.27 1.27)) (justify right))
     )
-    (property "Footprint" "Diode_THT:D_DO-41_SOD81_P10.16mm_Horizontal" (id 2) (at 313.055 140.97 0)
+    (property "Footprint" "Diode_THT:D_DO-41_SOD81_P10.16mm_Horizontal" (id 2) (at 325.755 149.86 0)
       (effects (font (size 1.27 1.27)) hide)
     )
-    (property "Datasheet" "http://www.vishay.com/docs/88503/1n4001.pdf" (id 3) (at 308.61 140.97 0)
+    (property "Datasheet" "http://www.vishay.com/docs/88503/1n4001.pdf" (id 3) (at 321.31 149.86 0)
       (effects (font (size 1.27 1.27)) hide)
     )
@@
       (reference "JP1") (unit 1) (value "O2 HEAT ENABLE") (footprint "")
     )
+    (path "/56a69039-9b11-4de5-b2fa-d809e1c0b553"
+      (reference "JP?") (unit 1) (value "SolderJumper_2_Open") (footprint "")
+    )
     (path "/8c433e22-638c-4567-adb7-47aebdc28b4c"

Commit message: Change to regular jumper instead of solder jumper
Parts:
- removed JP?: SolderJumper_2_Open, symbol Jumper:SolderJumper_2_Open
- added JP2: Jumper_2_Open, symbol Jumper:Jumper_2_Open
- renumbered D5 to D4, D4 to D5, U5 to U4, U4 to U5
Connections:
- net at D4.1 (K), R26.1, R27.2: now also JP2.2 (B)
- net at D5.1 (K): now also JP2.1 (A)
Other:
- note added: "Oxygen Sensor"
- moved on the sheet: JP1

Commit message: Added footprints
Parts:
- removed R1: 27, symbol Device:R_Small
- removed R2: 1M, symbol Device:R_Small
- removed Y1: 16 mhz, symbol Device:Crystal_GND3_Small
- added R?: 1M, Resistor_SMD:R_0805_2012Metric_Pad1.20x1.40mm_HandSolder, symbol Device:R_Small
- added Y?: 16 mhz, Crystal:Resonator_SMD_Murata_CSTxExxV-3Pin_3.0x1.1mm_HandSoldering, symbol Device:Resonator_Small
- C1, C2, C21, C3, C5: value 100n -> 0.1uf; footprint (none) -> Capacitor_SMD:C_0805_2012Metric_Pad1.18x1.45mm_HandSolder
- C10: value 1n -> 1nf; footprint (none) -> Capacitor_SMD:C_0805_2012Metric_Pad1.18x1.45mm_HandSolder
- C11, C12, C13, C17, C18: value 0.22 uF -> 0.22uF; footprint (none) -> Capacitor_SMD:C_0805_2012Metric_Pad1.18x1.45mm_HandSolder
- C14, C15, C16, C7, C8, C9: value 0.1 uF -> 0.1uf; footprint (none) -> Capacitor_SMD:C_0805_2012Metric_Pad1.18x1.45mm_HandSolder
- C19: value 0.33 uF -> 0.33uF; footprint (none) -> Capacitor_SMD:C_0805_2012Metric_Pad1.18x1.45mm_HandSolder
- C20: value 10n -> 10nf; footprint (none) -> Capacitor_SMD:C_0805_2012Metric_Pad1.18x1.45mm_HandSolder
- C22, C27: value 1u -> 1uf; footprint (none) -> Capacitor_SMD:C_0805_2012Metric_Pad1.18x1.45mm_HandSolder
- C23: value 10u -> 10uf; footprint Capacitors_THT:CP_Radial_Tantal_D6.0mm_P2.50mm -> Capacitor_THT:CP_Radial_Tantal_D6.0mm_P2.50mm
- C26: value 47u -> 47uf
- C4: footprint (none) -> Capacitor_SMD:C_0805_2012Metric_Pad1.18x1.45mm_HandSolder
- C6: value 0.1u -> 0.1uf; footprint (none) -> Capacitor_SMD:C_0805_2012Metric_Pad1.18x1.45mm_HandSolder
- J2: footprint (none) -> Connector_PinHeader_2.54mm:PinHeader_2x03_P2.54mm_Vertical
- J3: footprint (none) -> Connector_PinHeader_2.54mm:PinHeader_1x06_P2.54mm_Vertical
- JP1: footprint (none) -> Connector_PinHeader_2.54mm:PinHeader_1x03_P2.54mm_Vertical
- JP2: footprint (none) -> Connector_PinHeader_2.54mm:PinHeader_1x02_P2.54mm_Vertical
- LED1, LED2, LED3, LED4: footprint (none) -> LED_SMD:LED_0805_2012Metric_Pad1.15x1.40mm_HandSolder; p/n (none) -> 150080VS75000
- R1: renamed from R3; footprint (none) -> Resistor_SMD:R_0805_2012Metric_Pad1.20x1.40mm_HandSolder
- R10: renamed from R12; value 3.9K -> 3.9k; footprint (none) -> Resistor_SMD:R_0805_2012Metric_Pad1.20x1.40mm_HandSolder
- R11: renamed from R13; value 1K -> 1k; footprint (none) -> Resistor_SMD:R_0805_2012Metric_Pad1.20x1.40mm_HandSolder
- R12: renamed from R14; value 470 -> 470k; footprint (none) -> Resistor_SMD:R_0805_2012Metric_Pad1.20x1.40mm_HandSolder
- R13: renamed from R15; value 470 -> 470k; footprint (none) -> Resistor_SMD:R_0805_2012Metric_Pad1.20x1.40mm_HandSolder
- R14: renamed from R16; value 470 -> 470k; footprint (none) -> Resistor_SMD:R_0805_2012Metric_Pad1.20x1.40mm_HandSolder
- R15: renamed from R17; footprint (none) -> Resistor_SMD:R_0805_2012Metric_Pad1.20x1.40mm_HandSolder
- R16: renamed from R18; footprint (none) -> Resistor_SMD:R_0805_2012Metric_Pad1.20x1.40mm_HandSolder
- R17: renamed from R19; footprint (none) -> Resistor_SMD:R_0805_2012Metric_Pad1.20x1.40mm_HandSolder
- R18: renamed from R20; footprint (none) -> Resistor_SMD:R_0805_2012Metric_Pad1.20x1.40mm_HandSolder
- R19: renamed from R21; footprint (none) -> Resistor_SMD:R_0805_2012Metric_Pad1.20x1.40mm_HandSolder
- R2: renamed from R4; footprint (none) -> Resistor_SMD:R_0805_2012Metric_Pad1.20x1.40mm_HandSolder
- R20: renamed from R22; footprint (none) -> Resistor_SMD:R_0805_2012Metric_Pad1.20x1.40mm_HandSolder
- R21: renamed from R23; footprint (none) -> Resistor_SMD:R_0805_2012Metric_Pad1.20x1.40mm_HandSolder
- R22: renamed from R24; footprint (none) -> Resistor_SMD:R_0805_2012Metric_Pad1.20x1.40mm_HandSolder
- R23: renamed from R25; footprint (none) -> Resistor_SMD:R_0805_2012Metric_Pad1.20x1.40mm_HandSolder
- R24: renamed from R26; footprint (none) -> Resistor_SMD:R_0805_2012Metric_Pad1.20x1.40mm_HandSolder
- R25: renamed from R27; footprint (none) -> Resistor_SMD:R_0805_2012Metric_Pad1.20x1.40mm_HandSolder
- R26: renamed from R28; footprint (none) -> Resistor_SMD:R_0805_2012Metric_Pad1.20x1.40mm_HandSolder
- R27: renamed from R29; footprint (none) -> Resistor_SMD:R_0805_2012Metric_Pad1.20x1.40mm_HandSolder
- R28: renamed from R30; footprint (none) -> Resistor_SMD:R_0805_2012Metric_Pad1.20x1.40mm_HandSolder
- R29: renamed from R31; footprint (none) -> Resistor_SMD:R_0805_2012Metric_Pad1.20x1.40mm_HandSolder
- R3: renamed from R5; value 2.49K -> 2.49k; footprint (none) -> Resistor_SMD:R_0805_2012Metric_Pad1.20x1.40mm_HandSolder
- R30: renamed from R32; footprint (none) -> Resistor_SMD:R_0805_2012Metric_Pad1.20x1.40mm_HandSolder
- R31: renamed from R33; footprint (none) -> Resistor_SMD:R_0805_2012Metric_Pad1.20x1.40mm_HandSolder
- R32: renamed from R34; footprint (none) -> Resistor_SMD:R_0805_2012Metric_Pad1.20x1.40mm_HandSolder
- R33: renamed from R35; footprint (none) -> Resistor_SMD:R_0805_2012Metric_Pad1.20x1.40mm_HandSolder
- R34: renamed from R36; footprint (none) -> Resistor_THT:R_Axial_DIN0207_L6.3mm_D2.5mm_P5.08mm_Vertical
- R4: renamed from R6; value 2.49K -> 2.49k; footprint (none) -> Resistor_SMD:R_0805_2012Metric_Pad1.20x1.40mm_HandSolder
- R5: renamed from R7; footprint (none) -> Resistor_SMD:R_0805_2012Metric_Pad1.20x1.40mm_HandSolder
- R6: renamed from R8; footprint (none) -> Resistor_SMD:R_0805_2012Metric_Pad1.20x1.40mm_HandSolder
- R7: renamed from R9; value 470 -> 470k; footprint (none) -> Resistor_SMD:R_0805_2012Metric_Pad1.20x1.40mm_HandSolder
- R8: renamed from R10; value 470 -> 470k; footprint (none) -> Resistor_SMD:R_0805_2012Metric_Pad1.20x1.40mm_HandSolder
- R9: renamed from R11; value 470 -> 470k; footprint (none) -> Resistor_SMD:R_0805_2012Metric_Pad1.20x1.40mm_HandSolder
- U3: value ERZ -> ERZ-V14D220
- U4: value LM2940T-5.0 -> LM340T-5.0
- U5: value 74LS02 -> 74LS02DR; footprint (none) -> Package_SO:SOIC-14_3.9x8.7mm_P1.27mm
- U6: value 74LS14 -> 74LS14DR; footprint Package_DIP:DIP-14_W7.62mm -> Package_SO:SOIC-14_3.9x8.7mm_P1.27mm
Connections:
- net +5V: now also Y?.2
- net at U1.33 (XTAL2): now also R?.2, Y?.3
- net at U1.34 (XTAL1): now also R?.1, Y?.1
Other:
- moved on the sheet: C5

Commit message: begin PCB routing
Parts:
- removed D3: 1N4004, Diode_THT:D_DO-41_SOD81_P10.16mm_Horizontal, symbol Diode:1N4004
- removed LED2: GREEN, LED_SMD:LED_0805_2012Metric_Pad1.15x1.40mm_HandSolder, symbol Device:LED
- removed R17: 2k, Resistor_SMD:R_0805_2012Metric_Pad1.20x1.40mm_HandSolder, symbol Device:R_Small
- C24, C25: footprint Capacitors_THT:C_Disc_D3.8mm_W2.6mm_P2.50mm -> Capacitor_THT:C_Disc_D3.8mm_W2.6mm_P2.50mm
- C26: footprint Capacitors_THT:CP_Radial_Tantal_D6.0mm_P2.50mm -> Capacitor_THT:CP_Radial_Tantal_D6.0mm_P2.50mm
- J1: value Main Connector -> Conn_02x18_Top_Bottom; footprint Connector_JAE:JAE_LY20-36P-DLT1_2x18_P2.00mm_Horizontal -> Connector_PinHeader_2.54mm:PinHeader_2x18_P2.54mm_Vertical
- U2: footprint 21-0061L_MXM -> Package_SO:MSOP-10_3x3mm_P0.5mm
- U3: footprint Varistors:RV_Disc_D15.5_W4.2_P7.5 -> Varistor:RV_Disc_D7mm_W3.4mm_P5mm
- U4: footprint TO_SOT_Packages_THT:TO-220_Vertical -> Package_TO_SOT_THT:TO-220-3_Vertical
- U7: footprint Package_DIP:DIP-8-N6_W7.62mm -> Package_DIP:DIP-8_W7.62mm
- gave numbers to parts that had none: 2
- renumbered R9 to R10, R10 to R11, R11 to R12, R12 to R13, R13 to R14, R14 to R15, R15 to R16, R16 to R17, R18 to R19, R1 to R2, R19 to R20, R20 to R21, R21 to R22, R22 to R23, R23 to R24, R24 to R25, R25 to R26, R26 to R27, R27 to R28, R28 to R29, R2 to R3, R29 to R30, R30 to R31, R31 to R32, R32 to R33, R33 to R34, R34 to R35, R3 to R4, R4 to R5, R5 to R6, R6 to R7, R7 to R8, R8 to R9
Connections:
- net FAN_RELAY is gone; now on net FAN RELAY: D7.1 (K), Q4.2 (D)
- net FP_RELAY is gone; now on net FP RELAY: Q2.2 (D)
- net +12V: now also J1.19 (Pin_19); no longer J1.1 (Pin_1)
- net +5V: now also J1.31 (Pin_31); no longer C1.2, C11.2, C12.2, C13.2, C14.2, C15.2, C16.2, C17.2, C18.2, C19.2, C2.2, C20.2, C21.2, C22.2, C27.2, C3.2, C4.2, C5.2, C7.2, C8.2, C9.2, J1.10 (Pin_10), J1.13 (Pin_13), J1.24 (Pin_24), J1.35 (Pin_35), J1.36 (Pin_36), J1.8 (Pin_8), J2.6 (Pin_6), J3.1 (Pin_1), J3.2 (Pin_2), JP1.1 (A), LED4.1 (K), Q1.3 (S), Q2.3 (S), Q3.1 (S), Q3.3 (1), Q4.3 (S), R12.1, R19.2, R20.2, R25.2, R28.2, R30.2, R31.2, U1.11 (GND), U1.32 (GND), U1.62 (GND), U1.81 (GND), U1.99 (GND), U2.4 (BIAS), U2.5 (GND), U2.6 (ZERO_EN), U2.9 (INT_THRS), U5.7 (GND), U6.7 (GND), U7.4 (GND), U7.5 (GND), Y1.2
- net +BATT: now also J1.1 (Pin_1); no longer J1.19 (Pin_19)
- net AIR VALVE: now also J1.12 (Pin_12); no longer J1.30 (Pin_30)
- net ARDUINO-D3: now also J1.5 (Pin_5); no longer J1.23 (Pin_23)
- net CHECK ENGINE: now also J1.3 (Pin_3); no longer J1.21 (Pin_21)
- net CKP +: now also J1.21 (Pin_21); no longer J1.3 (Pin_3)
- net CKP -: now also J1.27 (Pin_27); no longer J1.9 (Pin_9)
- net CLT: now also J1.4 (Pin_4); no longer J1.22 (Pin_22)
- net CLUTCH SW: now also J1.30 (Pin_30); no longer J1.12 (Pin_12)
- net Earth: no longer C23.2, C24.2, C25.2, C26.2, D6.2 (A), U3.2, U4.2 (GND)
- net FAN RELAY: now also J1.15 (Pin_15); no longer J1.33 (Pin_33)
- net FP RELAY: now also J1.29 (Pin_29); no longer J1.11 (Pin_11)
- net IAT: now also J1.7 (Pin_7); no longer J1.25 (Pin_25)
- net IGN: now also J1.36 (Pin_36); no longer J1.18 (Pin_18)
- net INJECTOR: now also J1.34 (Pin_34); no longer J1.16 (Pin_16)
- net KICKSTAND SW: now also J1.11 (Pin_11); no longer J1.29 (Pin_29)
- net KILL SW: now also J1.16 (Pin_16); no longer J1.34 (Pin_34)
- net MAP: now also J1.24 (Pin_24); no longer J1.6 (Pin_6)
- net NEUTRAL SW: now also J1.2 (Pin_2); no longer J1.20 (Pin_20)
- net O2S +: now also J1.25 (Pin_25); no longer J1.7 (Pin_7)
- net O2S HEAT +: now also J1.35 (Pin_35); no longer J1.17 (Pin_17)
- net SPEED: now also J1.8 (Pin_8); no longer J1.26 (Pin_26)
- net SUB A +: now also J1.33 (Pin_33); no longer J1.15 (Pin_15)
- net SUB A -: now also J1.13 (Pin_13); no longer J1.31 (Pin_31)
- net SUB B +: now also J1.32 (Pin_32); no longer J1.14 (Pin_14)
- net SUB B -: now also J1.14 (Pin_14); no longer J1.32 (Pin_32)
- net SUB TPS: now also J1.9 (Pin_9); no longer J1.27 (Pin_27)
- net TEMP WARN: now also J1.10 (Pin_10); no longer J1.28 (Pin_28)
- net TPS: now also J1.23 (Pin_23); no longer J1.5 (Pin_5)
- net Vehicle Down: now also J1.20 (Pin_20); no longer J1.2 (Pin_2)
- new net GND: C1.2, C11.2, C12.2, C13.2, C14.2, C15.2, C16.2, C17.2, C18.2, C19.2, C2.2, C20.2, C21.2, C22.2, C23.2, C24.2, C25.2, C26.2, C27.2, C3.2, C4.2, C5.2, C7.2, C8.2, C9.2, D6.2 (A), J1.17 (Pin_17), J1.18 (Pin_18), J1.26 (Pin_26), J1.28 (Pin_28), J1.6 (Pin_6), J2.6 (Pin_6), J3.1 (Pin_1), J3.2 (Pin_2), JP1.1 (A), LED4.1 (K), Q1.3 (S), Q2.3 (S), Q3.1 (S), Q3.3 (1), Q4.3 (S), R12.1, R19.2, R20.2, R25.2, R28.2, R30.2, R31.2, U1.11 (GND), U1.32 (GND), U1.62 (GND), U1.81 (GND), U1.99 (GND), U2.4 (BIAS), U2.5 (GND), U2.6 (ZERO_EN), U2.9 (INT_THRS), U3.2, U4.2 (GND), U5.7 (GND), U6.7 (GND), U7.4 (GND), U7.5 (GND), Y1.2
