File: klxecu.kicad_sch (KiCad schematic)
At the start: 88 parts, among them IC1 SP721, J1 Conn_02x18_Top_Bottom, J2 ICSP, J3 Arduino Comms Header, Q1 STP62NS04Z, Q2 STP62NS04Z, Q3 IRF7301PBF, Q4 STP62NS04Z, U1 ATmega2560-16A, U2 MAX9924UAUB+, U3 ERZ-V14D220, U4 LM340T-5.0, U5 74LS02DR, U6 74LS14DR, U7 TC4422AVPA, Y1 16 mhz

Commit message: Updates
Parts:
- removed C1, C2, C3, C5, C6: 0.1uf, Capacitor_SMD:C_0805_2012Metric_Pad1.18x1.45mm_HandSolder, symbol Device:C_Small
- removed C4: 22pf, Capacitor_SMD:C_0805_2012Metric_Pad1.18x1.45mm_HandSolder, symbol Device:C_Small
- removed D4, D5, D7: 1N4004, Diode_THT:D_DO-41_SOD81_P10.16mm_Horizontal, symbol Diode:1N4004
- removed J2: ICSP, Connector_PinHeader_2.54mm:PinHeader_2x03_P2.54mm_Vertical, symbol Connector_Generic:Conn_02x03_Odd_Even
- removed J3: Arduino Comms Header, Connector_PinHeader_2.54mm:PinHeader_1x06_P2.54mm_Vertical, symbol Connector:Conn_01x06_Male
- removed JP2: Jumper_2_Open, Connector_PinHeader_2.54mm:PinHeader_1x02_P2.54mm_Vertical, symbol Jumper:Jumper_2_Open
- removed LED3: GREEN, LED_SMD:LED_0805_2012Metric_Pad1.15x1.40mm_HandSolder, symbol Device:LED
- removed Q3: IRF7301PBF, Package_SO:SOIC-8_3.9x4.9mm_P1.27mm, symbol Transistor_FET:IRF7309IPBF
- removed R1: 1M, Resistor_SMD:R_0805_2012Metric_Pad1.20x1.40mm_HandSolder, symbol Device:R_Small
- removed R29: 2k, Resistor_SMD:R_0805_2012Metric_Pad1.20x1.40mm_HandSolder, symbol Device:R_Small
- removed U1: ATmega2560-16A, Package_QFP:TQFP-100_14x14mm_P0.5mm, symbol MCU_Microchip_ATmega:ATmega2560-16A
- removed U5: 74LS02DR, Package_SO:SOIC-14_3.9x8.7mm_P1.27mm, symbol 74xx:74LS02
- removed Y1: 16 mhz, Crystal:Resonator_SMD_Murata_CSTxExxV-3Pin_3.0x1.1mm_HandSoldering, symbol Device:Resonator_Small
- added A1: Pololu_Breakout_A4988, Module:Pololu_Breakout-16_15.2x20.3mm, symbol Driver_Motor:Pololu_Breakout_A4988
- added C11: 0.22uF, Capacitor_SMD:C_0805_2012Metric_Pad1.18x1.45mm_HandSolder, symbol Device:C_Small
- added C19: 100uf, Capacitor_THT:CP_Radial_D5.0mm_P2.50mm, symbol Device:C_Polarized_Small
- added C8: 0.1uf, Capacitor_SMD:C_0805_2012Metric_Pad1.18x1.45mm_HandSolder, symbol Device:C_Small
- added J1: Conn_02x20_Odd_Even, Connector_PinSocket_2.54mm:PinSocket_2x20_P2.54mm_Vertical, symbol Connector_Generic:Conn_02x20_Odd_Even
- added J3: Conn_02x16_Odd_Even, Connector_PinSocket_2.54mm:PinSocket_2x16_P2.54mm_Vertical, symbol Connector_Generic:Conn_02x16_Odd_Even
- added JP2: Jumper_3_Open, Connector_PinHeader_2.54mm:PinHeader_1x03_P2.54mm_Vertical, symbol Jumper:Jumper_3_Open
- added Q3, Q4: STP62NS04Z, Package_TO_SOT_THT:TO-220-3_Vertical, symbol Transistor_FET:BUZ11
- added R10: 470, Resistor_THT:R_Axial_DIN0207_L6.3mm_D2.5mm_P5.08mm_Vertical, symbol Device:R_Small
- added U2: ATtiny84-20P, Package_DIP:DIP-14_W7.62mm, symbol MCU_Microchip_ATtiny:ATtiny84-20P
- R1: renamed from R2; footprint Resistor_SMD:R_0805_2012Metric_Pad1.20x1.40mm_HandSolder -> Resistor_THT:R_Axial_DIN0207_L6.3mm_D2.5mm_P5.08mm_Vertical
- R11, R12, R16, R17: footprint Resistor_SMD:R_0805_2012Metric_Pad1.20x1.40mm_HandSolder -> Resistor_THT:R_Axial_DIN0207_L6.3mm_D2.5mm_P5.08mm_Vertical
- R13, R14, R15: value 470k -> 470; footprint Resistor_SMD:R_0805_2012Metric_Pad1.20x1.40mm_HandSolder -> Resistor_THT:R_Axial_DIN0207_L6.3mm_D2.5mm_P5.08mm_Vertical
- R18: renamed from R19; footprint Resistor_SMD:R_0805_2012Metric_Pad1.20x1.40mm_HandSolder -> Resistor_THT:R_Axial_DIN0207_L6.3mm_D2.5mm_P5.08mm_Vertical
- R19: renamed from R20; footprint Resistor_SMD:R_0805_2012Metric_Pad1.20x1.40mm_HandSolder -> Resistor_THT:R_Axial_DIN0207_L6.3mm_D2.5mm_P5.08mm_Vertical
- R2: renamed from R3; footprint Resistor_SMD:R_0805_2012Metric_Pad1.20x1.40mm_HandSolder -> Resistor_THT:R_Axial_DIN0207_L6.3mm_D2.5mm_P5.08mm_Vertical
- R20: renamed from R21; footprint Resistor_SMD:R_0805_2012Metric_Pad1.20x1.40mm_HandSolder -> Resistor_THT:R_Axial_DIN0207_L6.3mm_D2.5mm_P5.08mm_Vertical
- R21: renamed from R22; footprint Resistor_SMD:R_0805_2012Metric_Pad1.20x1.40mm_HandSolder -> Resistor_THT:R_Axial_DIN0207_L6.3mm_D2.5mm_P5.08mm_Vertical
- R22: renamed from R25; footprint Resistor_SMD:R_0805_2012Metric_Pad1.20x1.40mm_HandSolder -> Resistor_THT:R_Axial_DIN0207_L6.3mm_D2.5mm_P5.08mm_Vertical
- R23: renamed from R26; footprint Resistor_SMD:R_0805_2012Metric_Pad1.20x1.40mm_HandSolder -> Resistor_THT:R_Axial_DIN0207_L6.3mm_D2.5mm_P5.08mm_Vertical
- R24: renamed from R27; footprint Resistor_SMD:R_0805_2012Metric_Pad1.20x1.40mm_HandSolder -> Resistor_THT:R_Axial_DIN0207_L6.3mm_D2.5mm_P5.08mm_Vertical
- R25: renamed from R28; footprint Resistor_SMD:R_0805_2012Metric_Pad1.20x1.40mm_HandSolder -> Resistor_THT:R_Axial_DIN0207_L6.3mm_D2.5mm_P5.08mm_Vertical
- R26: renamed from R23; footprint Resistor_SMD:R_0805_2012Metric_Pad1.20x1.40mm_HandSolder -> Resistor_THT:R_Axial_DIN0207_L6.3mm_D2.5mm_P5.08mm_Vertical
- R27: renamed from R24; footprint Resistor_SMD:R_0805_2012Metric_Pad1.20x1.40mm_HandSolder -> Resistor_THT:R_Axial_DIN0207_L6.3mm_D2.5mm_P5.08mm_Vertical
- R28: renamed from R30; footprint Resistor_SMD:R_0805_2012Metric_Pad1.20x1.40mm_HandSolder -> Resistor_THT:R_Axial_DIN0207_L6.3mm_D2.5mm_P5.08mm_Vertical
- R29: renamed from R31; footprint Resistor_SMD:R_0805_2012Metric_Pad1.20x1.40mm_HandSolder -> Resistor_THT:R_Axial_DIN0207_L6.3mm_D2.5mm_P5.08mm_Vertical
- R3: renamed from R4; footprint Resistor_SMD:R_0805_2012Metric_Pad1.20x1.40mm_HandSolder -> Resistor_THT:R_Axial_DIN0207_L6.3mm_D2.5mm_P5.08mm_Vertical
- R30: renamed from R32; footprint Resistor_SMD:R_0805_2012Metric_Pad1.20x1.40mm_HandSolder -> Resistor_THT:R_Axial_DIN0207_L6.3mm_D2.5mm_P5.08mm_Vertical
- R31: renamed from R33; footprint Resistor_SMD:R_0805_2012Metric_Pad1.20x1.40mm_HandSolder -> Resistor_THT:R_Axial_DIN0207_L6.3mm_D2.5mm_P5.08mm_Vertical
- R32: renamed from R34; footprint Resistor_SMD:R_0805_2012Metric_Pad1.20x1.40mm_HandSolder -> Resistor_THT:R_Axial_DIN0207_L6.3mm_D2.5mm_P5.08mm_Vertical
- R4: renamed from R6; footprint Resistor_SMD:R_0805_2012Metric_Pad1.20x1.40mm_HandSolder -> Resistor_THT:R_Axial_DIN0207_L6.3mm_D2.5mm_P5.08mm_Vertical
- R5: renamed from R7; footprint Resistor_SMD:R_0805_2012Metric_Pad1.20x1.40mm_HandSolder -> Resistor_THT:R_Axial_DIN0207_L6.3mm_D2.5mm_P5.08mm_Vertical
- R6: renamed from R5; footprint Resistor_SMD:R_0805_2012Metric_Pad1.20x1.40mm_HandSolder -> Resistor_THT:R_Axial_DIN0207_L6.3mm_D2.5mm_P5.08mm_Vertical
- R7: renamed from R8; footprint Resistor_SMD:R_0805_2012Metric_Pad1.20x1.40mm_HandSolder -> Resistor_THT:R_Axial_DIN0207_L6.3mm_D2.5mm_P5.08mm_Vertical
- R8: renamed from R9; value 470k -> 470
- R9: renamed from R10; value 470k -> 470; footprint Resistor_SMD:R_0805_2012Metric_Pad1.20x1.40mm_HandSolder -> Resistor_THT:R_Axial_DIN0207_L6.3mm_D2.5mm_P5.08mm_Vertical
- renumbered C7 to C1, C15 to C10, C16 to C12, C17 to C13, C18 to C14, C19 to C15, C20 to C16, C21 to C17, C22 to C18, C10 to C2, C27 to C20, C23 to C21, C24 to C22, C25 to C23, C26 to C24, C8 to C3, C9 to C4, C11 to C5, C12 to C6, C13 to C7, C14 to C9, D2 to D1, D1 to D3, D6 to D4, J1 to J2, LED4 to LED2, Q4 to Q5, R35 to R33, U2 to U1, U6 to U3, U7 to U4, U3 to U5, U4 to U6
Connections:
- net Earth is gone; now on net GND: IC1.4 (P4)
- net +5V: now also A1.2 (VDD), J1.5 (Pin_5), J1.6 (Pin_6), JP2.1 (A), U2.1 (VCC), U2.4 (~{RESET}/PB3)
- net +BATT: now also C19.1, JP2.3 (B)
- net ARDUINO-A0: now also J3.1 (Pin_1)
- net ARDUINO-A1: now also J3.2 (Pin_2)
- net ARDUINO-A2: now also J3.3 (Pin_3)
- net ARDUINO-A3: now also J3.4 (Pin_4)
- net ARDUINO-A4: now also J3.5 (Pin_5)
- net ARDUINO-A5: now also J3.6 (Pin_6)
- net ARDUINO-D19: now also J1.28 (Pin_28)
- net ARDUINO-D23: now also J1.32 (Pin_32)
- net ARDUINO-D4: now also J1.13 (Pin_13)
- net ARDUINO-D5: now also J1.14 (Pin_14)
- net ARDUINO-D6: now also J1.15 (Pin_15), U2.5 (PB2)
- net ARDUINO-D7: now also J1.16 (Pin_16)
- net ARDUINO-D8: now also J1.17 (Pin_17), J1.18 (Pin_18)
- net ARDUINO-RST: now also J1.8 (Pin_8), U2.3 (XTAL2/PB1)
- net CHECK ENGINE: now also Q3.2 (D)
- net GND: now also A1.1 (GND), A1.7 (GND), C11.2, C19.2, C8.2, J1.3 (Pin_3), J1.4 (Pin_4), Q3.3 (S), Q4.3 (S), U2.14 (GND)
- net SUB A +: now also A1.4 (1A)
- net SUB A -: now also A1.3 (1B)
- net SUB B +: now also A1.5 (2A)
- net SUB B -: now also A1.6 (2B)
- net SUB TPS: now also C8.1, R10.1
- net TEMP WARN: now also Q4.2 (D)
- net ATTINY-D10: now reaches R22.1, R23.2
- net ATTINY-D10: now also U2.2 (XTAL1/PB0)
- net ATTINY-A4: now reaches U3.6
- net ATTINY-A4: now also U2.9 (PA4)
- net at R31.1: now also Q4.1 (G)
- net at R23.1: now also Q3.1 (G)
- net ATTINY-A2: now reaches U3.2
- net ATTINY-A2: now also U2.11 (PA2)
- net ATTINY-A3: now reaches U3.4
- net ATTINY-A3: now also U2.10 (PA3)
- new net: A1.8 (VMOT), JP2.2 (C)
- new net: A1.16 (DIR), U2.7 (PA6)
- new net: A1.15 (STEP), U2.8 (PA5)
- new net: A1.13 (~{RESET}), A1.14 (~{SLEEP})
- new net ATTINY-A1: C11.1, R10.2, U2.12 (PA1)
- no-connect marks 2 -> 11
Other:
- note added: "Subthrottle Position Sensor"
- moved on the sheet: C16, C17, C18, C2, C21, C22, C23, C24, D3, D4, IC1, R16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
