File: klxecu.kicad_sch (KiCad schematic)
At the start: 80 parts, among them IC1 SP721, J1 Conn_02x20_Odd_Even, J2 Conn_02x18_Top_Bottom, J3 Conn_02x16_Odd_Even, Q1 STP62NS04Z, Q2 STP62NS04Z, Q3 STP62NS04Z, Q4 STP62NS04Z, Q5 STP62NS04Z, U1 MAX9924UAUB+, U2 ATtiny84-20P, U3 74LS14DR, U4 TC4422AVPA, U5 ERZ-V14D220, U6 LM340T-5.0

Commit message: Technically all the nets are connected
Connections:
- net CKP+ is gone; now on net CKP +: R2.1, R4.2
- net CKP- is gone; now on net CKP -: R2.2, R5.1
- net +12V: now also JP2.3 (B)
- net +BATT: no longer JP2.3 (B)
Changed lines of the file:
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@@
     )
   )
-  (global_label "CKP-" (shape input) (at 132.08 123.19 180) (fields_autoplaced)
-    (effects (font (size 1.27 1.27)) (justify right))
-    (property "Intersheet References" "${INTERSHEET_REFS}" (id 0) (at 124.2845 123.1106 0)
+  (global_label "CKP -" (shape input) (at 132.08 123.19 180) (fields_autoplaced)
+    (effects (font (size 1.27 1.27)) (justify right))
+    (property "Intersheet References" "${INTERSHEET_REFS}" (id 0) (at 123.3169 123.1106 0)
       (effects (font (size 1.27 1.27)) (justify right) hide)
     )
@@
     )
   )
-  (global_label "CKP+" (shape input) (at 132.08 118.11 180) (fields_autoplaced)
-    (effects (font (size 1.27 1.27)) (justify right))
-    (property "Intersheet References" "${INTERSHEET_REFS}" (id 0) (at 124.2845 118.1894 0)
+  (global_label "CKP +" (shape input) (at 132.08 118.11 180) (fields_autoplaced)
+    (effects (font (size 1.27 1.27)) (justify right))
+    (property "Intersheet References" "${INTERSHEET_REFS}" (id 0) (at 123.3169 118.0306 0)
       (effects (font (size 1.27 1.27)) (justify right) hide)
     )
@@
     (pin "1")
     (pin "2")
+  )
+  (symbol (lib_id "power:+12V") (at 273.05 196.85 0) (unit 1)
+    (in_bom yes) (on_board yes) (fields_autoplaced)
+    (property "Reference" "#PWR0102" (id 0) (at 273.05 200.66 0)
+      (effects (font (size 1.27 1.27)) hide)
+    )
+    (property "Value" "+12V" (id 1) (at 273.05 191.77 0))
+    (property "Footprint" "" (id 2) (at 273.05 196.85 0)
+      (effects (font (size 1.27 1.27)) hide)
+    )
+    (property "Datasheet" "" (id 3) (at 273.05 196.85 0)
+      (effects (font (size 1.27 1.27)) hide)
+    )
+    (pin "1")
   )
   (symbol (lib_id "Device:C_Small") (at 210.82 29.21 0) (unit 1)
@@
     )
     (property "Datasheet" "" (id 3) (at 193.04 256.54 0)
-      (effects (font (size 1.27 1.27)) hide)
-    )
-    (pin "1")
-  )
-  (symbol (lib_id "power:+BATT") (at 273.05 196.85 0) (unit 1)
-    (in_bom yes) (on_board yes) (fields_autoplaced)
-    (property "Reference" "#PWR027" (id 0) (at 273.05 200.66 0)
-      (effects (font (size 1.27 1.27)) hide)
-    )
-    (property "Value" "+BATT" (id 1) (at 273.05 191.77 0))
-    (property "Footprint" "" (id 2) (at 273.05 196.85 0)
-      (effects (font (size 1.27 1.27)) hide)
-    )
-    (property "Datasheet" "" (id 3) (at 273.05 196.85 0)
       (effects (font (size 1.27 1.27)) hide)
     )
@@
       (reference "#PWR026") (unit 1) (value "+5V") (footprint "")
     )
-    (path "/981343fd-6c2f-4f25-a633-b3f209534efd"
-      (reference "#PWR027") (unit 1) (value "+BATT") (footprint "")
-    )
     (path "/eb69b83d-87bd-4e80-a26a-e65f7546937d"
       (reference "#PWR028") (unit 1) (value "GND") (footprint "")
@@
       (reference "#PWR0101") (unit 1) (value "GND") (footprint "")
     )
+    (path "/0df6cb23-cf9f-4e1f-8aa1-c7034a9394f9"
+      (reference "#PWR0102") (unit 1) (value "+12V") (footprint "")
+    )
     (path "/ce94b8f1-b9c4-4ca5-9f9f-15aed9f37d84"

Commit message: Misc updates
- Add pin to handle cluch for launch control
- re-do PCB from scratch (more things go on the backside this time)
Parts:
- removed D1: 1N4004, Diode_THT:D_DO-41_SOD81_P10.16mm_Horizontal, symbol Diode:1N4004
- removed J2: Conn_02x18_Top_Bottom, Connector_PinHeader_2.54mm:PinHeader_2x18_P2.54mm_Vertical, symbol Connector_Generic:Conn_02x18_Top_Bottom
- removed JP1: O2 HEAT ENABLE, Connector_PinHeader_2.54mm:PinHeader_1x03_P2.54mm_Vertical, symbol Jumper:Jumper_3_Open
- removed LED1, LED2: GREEN, LED_SMD:LED_0805_2012Metric_Pad1.15x1.40mm_HandSolder, symbol Device:LED
- removed R1, R26, R27: 10k, Resistor_SMD:R_0805_2012Metric_Pad1.20x1.40mm_HandSolder, symbol Device:R_Small
- removed R14, R7, R8: 470, Resistor_SMD:R_0805_2012Metric_Pad1.20x1.40mm_HandSolder, symbol Device:R_Small
- removed R17, R32: 2k, Resistor_SMD:R_0805_2012Metric_Pad1.20x1.40mm_HandSolder, symbol Device:R_Small
- removed R18, R19, R22, R25, R28, R29: 100k, Resistor_SMD:R_0805_2012Metric_Pad1.20x1.40mm_HandSolder, symbol Device:R_Small
- removed R20, R21, R23, R24, R30, R31: 1k, Resistor_SMD:R_0805_2012Metric_Pad1.20x1.40mm_HandSolder, symbol Device:R_Small
- added J2: Conn_02x18_Odd_Even, Connector_PinHeader_2.54mm:PinHeader_2x18_P2.54mm_Vertical, symbol Connector_Generic:Conn_02x18_Odd_Even
- added J4: Conn_01x01_Male, Connector_PinHeader_2.54mm:PinHeader_1x01_P2.54mm_Vertical, symbol Connector:Conn_01x01_Male
- added Q1: 2N3904, Package_TO_SOT_THT:TO-92_Inline, symbol Transistor_BJT:2N3904
- added Q6: STP62NS04Z, Package_TO_SOT_THT:TO-220-3_Vertical, symbol Transistor_FET:BUZ11
- added R10: 10k, Resistor_SMD:R_0805_2012Metric, symbol Device:R_Small
- added R12: 1k, Resistor_SMD:R_0805_2012Metric_Pad1.20x1.40mm_HandSolder, symbol Device:R_Small
- added RN1: 470, Resistor_THT:R_Array_SIP12, symbol Device:R_Pack06_SIP_Split
- added RN2: 100k, Resistor_THT:R_Array_SIP6, symbol Device:R_Network05_Split
- added RN3: 1k, Resistor_THT:R_Array_SIP12, symbol Device:R_Pack06_SIP_Split
- added RN4: 10k, Resistor_THT:R_Array_SIP4, symbol Device:R_Network03_Split
- added unit 4 of U5
- R13: value 470 -> 100k
- R15, R9: value 470 -> 1k
- renumbered C21 to C1, C11 to C10, C7 to C11, C5 to C12, C14 to C13, C12 to C14, C3 to C15, C9 to C16, C15 to C17, C6 to C18, C13 to C19, C22 to C2, C16 to C20, C17 to C21, C18 to C22, C19 to C23, C20 to C24, C23 to C3, C24 to C4, C8 to C5, C2 to C6, C4 to C7, C1 to C8, C10 to C9, D3 to D1, D4 to D2, JP2 to JP1, Q1 to Q2, Q2 to Q3, Q5 to Q4, Q3 to Q5, Q4 to Q7, R2 to R1, R16 to R11, R33 to R14, R4 to R2, R5 to R3, R6 to R4, R10 to R5, R11 to R6, R12 to R7, R3 to R8, U5 to U1, U6 to U2, U1 to U3, U2 to U4, U3 to U5, U4 to U6
Connections:
- net +12V: now also R6.2, J2.2 (Pin_2), R10.2
- net +5V: now also J2.26 (Pin_26), RN4.1 (R1.1)
- net +BATT: now also J2.1 (Pin_1); no longer R6.2
- net AIR VALVE: now also J2.23 (Pin_23)
- net ARDUINO-A0: now also IC1.1 (P1), RN1.3 (R2.1); no longer IC1.5 (P5), R15.2
- net ARDUINO-A1: now also IC1.5 (P5), RN1.1 (R1.1); no longer IC1.6 (P6)
- net ARDUINO-A2: now also IC1.2 (P2), RN1.7 (R4.1); no longer IC1.7 (P7), R13.2
- net ARDUINO-A3: now also IC1.7 (P7), RN1.5 (R3.1); no longer IC1.1 (P1)
- net ARDUINO-A4: now also IC1.3 (P3), RN1.11 (R6.1); no longer IC1.2 (P2)
- net ARDUINO-A5: now also IC1.6 (P6), RN1.9 (R5.1); no longer IC1.3 (P3), R9.2
- net ARDUINO-D23: now also R12.1
- net ARDUINO-D4: now also RN2.3 (R2.2), RN3.3 (R2.1), RN3.5 (R3.1)
- net ARDUINO-D8: now also RN2.2 (R1.2), RN3.2 (R1.2)
- net ATTINY-D10: now also RN2.4 (R3.2), RN3.7 (R4.1)
- net CHECK ENGINE: now also J2.5 (Pin_5)
- net CKP +: now also J2.6 (Pin_6)
- net CKP -: now also J2.18 (Pin_18)
- net CLT: now also J2.7 (Pin_7), RN1.12 (R6.2)
- net CLUTCH SW: now also R15.2, J2.24 (Pin_24)
- net FAN RELAY: now also J2.29 (Pin_29)
- net FP RELAY: now also J2.22 (Pin_22)
- net GND: now also R13.2, J2.11 (Pin_11), J2.16 (Pin_16), J2.20 (Pin_20), J2.33 (Pin_33), J2.35 (Pin_35), Q1.1 (E), Q6.3 (S), RN2.1 (R1.1)
- net IAT: now also J2.13 (Pin_13), RN1.10 (R5.2); no longer R9.1
- net IGN: now also J2.36 (Pin_36)
- net INJECTOR: now also J2.32 (Pin_32)
- net KICKSTAND SW: now also J2.21 (Pin_21), RN4.3 (R2.2)
- net KILL SW: now also J2.31 (Pin_31)
- net MAP: now also J2.12 (Pin_12), RN1.4 (R2.2); no longer R15.1
- net NEUTRAL SW: now also J2.3 (Pin_3), RN4.2 (R1.2)
- net O2S +: now also J2.14 (Pin_14), RN1.8 (R4.2); no longer R13.1
- net O2S HEAT +: now also J2.34 (Pin_34), Q6.2 (D)
- net SPEED: now also J2.15 (Pin_15)
- net SUB A +: now also J2.30 (Pin_30)
- net SUB A -: now also J2.25 (Pin_25)
- net SUB B +: now also J2.28 (Pin_28)
- net SUB B -: now also J2.27 (Pin_27)
- net SUB TPS: now also J2.17 (Pin_17)
- net TEMP WARN: now also J2.19 (Pin_19)
- net TPS: now also J2.10 (Pin_10), RN1.6 (R3.2)
- net Vehicle Down: now also J2.4 (Pin_4)
- net ARDUINO-D32: now reaches J3.17 (Pin_17)
- net ARDUINO-D32: now also U4.5 (PB2)
- net ARDUINO-D34: now reaches J3.19 (Pin_19)
- net ARDUINO-D34: now also RN2.5 (R4.2), RN3.9 (R5.1)
- net ARDUINO-D38: now reaches J3.23 (Pin_23)
- net ARDUINO-D38: now also R9.2
- net ARDUINO-D42: now reaches J3.27 (Pin_27)
- net ARDUINO-D42: now also U5.8
- net at Q4.1 (G): now also RN3.12 (R6.2)
- net at C9.1, R6.1, R7.2: now also RN1.2 (R1.2)
- net at Q7.1 (G): now also RN3.10 (R5.2)
- net at Q5.1 (G): now also RN3.8 (R4.2)
- net at Q3.1 (G): now also RN3.4 (R2.2)
- net at U6.2 (INPUT): now also R13.1, R12.2
- net at Q2.1 (G): now also RN3.1 (R1.1)
- net at J1.19 (Pin_19): now also R15.1
- net ARDUINO-D30: now reaches J1.39 (Pin_39)
- net ARDUINO-D30: now also RN2.6 (R5.2), RN3.11 (R6.1)
- net ARDUINO-D3: no longer names the net of J1.12 (Pin_12)
- net ARDUINO-D5: no longer names the net of J1.14 (Pin_14)
- net ARDUINO-D6: no longer names the net of J1.15 (Pin_15)
- net ARDUINO-D6: no longer U4.5 (PB2)
- net ARDUINO-D7: no longer names the net of J1.16 (Pin_16)
- new net: J4.1 (Pin_1), Q1.3 (C), R10.1
- new net: Q6.1 (G), RN3.6 (R3.2)
- new net: Q1.2 (B), R9.1
- new net SELF DIAG: J2.9 (Pin_9), RN4.4 (R3.2), U5.9
Other:
- note added: "Safety Switches & Self-Diag"
- note added: "Tachometer Output"
- note removed: "Safety Switches"
- note removed: "Self Diagnosis"
- moved on the sheet: C1, C10, C12, C13, C14, C15, C16, C17, C18, C19, C2, C3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

Commit message: v1?
Parts:
- removed RN1: 470, Resistor_THT:R_Array_SIP12, symbol Device:R_Pack06_SIP_Split
- added R16, R17, R18, R19, R20, R21: 470, Resistor_SMD:R_0805_2012Metric_Pad1.20x1.40mm_HandSolder, symbol Device:R_Small
- added unit 6 of U5
- added unit 5 of U5
Connections:
- net +5V: now also U5.13
- net ARDUINO-A0: now also R19.2
- net ARDUINO-A1: now also R18.2
- net ARDUINO-A2: now also R21.2
- net ARDUINO-A3: now also R17.2
- net ARDUINO-A4: now also R20.2
- net ARDUINO-A5: now also R16.2
- net ARDUINO-D30: now also RN3.7 (R4.1); no longer RN3.11 (R6.1)
- net ATTINY-D10: now also RN3.11 (R6.1); no longer RN3.7 (R4.1)
- net CLT: now also R20.1
- net GND: now also U5.11
- net IAT: now also R16.1
- net MAP: now also R19.1
- net O2S +: now also R21.1
- net TPS: now also R17.1
- net at RN3.8 (R4.2): now also Q4.1 (G); no longer Q5.1 (G)
- net at RN3.12 (R6.2): now also Q5.1 (G); no longer Q4.1 (G)
- net at C9.1, R6.1, R7.2: now also R18.1
- no-connect marks 11 -> 13
Other:
- moved on the sheet: RN3D, RN3E, RN3F, U5G

Commit message: add gerber files
Parts:
- C1: value 10uf -> 10uF
- C14, C15, C16, C21, C5, C7, C8, C9: value 0.1uf -> 100nF
- C2, C3: value u1 -> 100nF
- C20: value 10nf -> 10nF
- C22, C24: value 1uf -> 1uF
- C23: value 100uf -> 100uF
- C4: value 47uf -> 47uF
- C6: value 1nf -> 1nF; LCSC (none) -> C46653
- R1: value 4.7k -> 4.7K
- R10, R2, R3, RN4: value 10k -> 10K
- R11, R12, R15, R7, R9, RN3: value 1k -> 1K
- R13, RN2: value 100k -> 100K
- R4, R8: value 2.49k -> 2.49K
- R6: value 3.9k -> 3.9K
