File: v2/klxecu.kicad_sch (KiCad schematic)
At the start: 65 parts, among them IC1 SP721, J1 Conn_01x02, J2 Conn_02x04_Counter_Clockwise, J3 Conn_01x01_Male, Q1 SSM3K357R, Q2 STP62NS04Z, Q3 SSM3K357R, Q4 SSM3K357R, Q5 SSM3K357R, Q6 STP62NS04Z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

Commit message: Changed to hierarchy of sheets
Parts:
- removed C10, C11, C12, C17, C18, C9: 0.22uF, Capacitor_SMD:C_0805_2012Metric_Pad1.18x1.45mm_HandSolder, symbol Device:C_Small
- removed C13, C14, C15, C5, C6, C7, C8: 100nF, Capacitor_SMD:C_0805_2012Metric_Pad1.18x1.45mm_HandSolder, symbol Device:C_Small
- removed C16: 0.33uF, Capacitor_SMD:C_0805_2012Metric_Pad1.18x1.45mm_HandSolder, symbol Device:C_Small
- removed C19: 0.1uf, Capacitor_SMD:C_0805_2012Metric, symbol Device:C_Small
- removed C21: 1uF, Capacitor_SMD:C_0805_2012Metric_Pad1.18x1.45mm_HandSolder, symbol Device:C_Small
- removed C?: 0.1uF, symbol Device:C_Small
- removed D2, D4: 1N5158, Diode_THT:D_DO-41_SOD81_P7.62mm_Horizontal, symbol Device:D_Schottky
- removed IC1: SP721, Package_DIP:DIP-8_W7.62mm, symbol modules:DIL8
- removed J2: Conn_02x04_Counter_Clockwise, mega_2560:vr_conditioner, symbol Connector_Generic:Conn_02x04_Counter_Clockwise
- removed J3: Conn_01x01_Male, Connector_PinHeader_2.54mm:PinHeader_1x01_P2.54mm_Vertical, symbol Connector:Conn_01x01_Male
- removed Q1, Q3, Q4, Q5, Q7: SSM3K357R, Package_TO_SOT_SMD:SOT-23, symbol Transistor_FET:2N7002
- removed Q2, Q6: STP62NS04Z, Package_TO_SOT_THT:TO-220-3_Vertical, symbol Transistor_FET:BUZ11
- removed R1, R8: 2.49K, Resistor_SMD:R_0805_2012Metric_Pad1.20x1.40mm_HandSolder, symbol Device:R_Small
- removed R10, R11, R4, R5, R6, R7, R9: 470, Resistor_SMD:R_0805_2012Metric_Pad1.20x1.40mm_HandSolder, symbol Device:R_Small
- removed R13: 1k, Resistor_SMD:R_0805_2012Metric_Pad1.20x1.40mm_HandSolder, symbol Device:R_Small
- removed R14: 10K, Resistor_SMD:R_0805_2012Metric, symbol Device:R_Small
- removed R15: 100K, Resistor_SMD:R_0805_2012Metric, symbol Device:R_Small
- removed R16: 1K, Resistor_SMD:R_0805_2012Metric, symbol Device:R_Small
- removed R17, R3: 1K, Resistor_SMD:R_0805_2012Metric_Pad1.20x1.40mm_HandSolder, symbol Device:R_Small
- removed R18: 100K, Resistor_SMD:R_0805_2012Metric_Pad1.20x1.40mm_HandSolder, symbol Device:R_Small
- removed R19: 47 2w, Resistor_THT:R_Axial_DIN0207_L6.3mm_D2.5mm_P5.08mm_Vertical, symbol Device:R_Small
- removed R2: 3.9K, Resistor_SMD:R_0805_2012Metric_Pad1.20x1.40mm_HandSolder, symbol Device:R_Small
- removed RN?: 10k, Resistor_THT:R_Array_SIP4, symbol Device:R_Network03
- removed U7: TC4422AVPA, Package_DIP:DIP-8_W7.62mm, symbol Driver_FET:TC4422
- removed U?: 74xx14, symbol mega_2560:74xx14
- J1: value Conn_01x02 -> CAM_SENSOR_IN
- U1: value mega_2560_pro -> Arduino Mega 2560 Pro
Connections:
- net DIR-ATTINY-A6: now reaches A1.16 (DIR), U5.7 (PA6)
- net STEP-ATTINY-A5: now reaches A1.15 (STEP), U5.8 (PA5)
- no-connect marks 14 -> 12
Other:
- added sheet Inputs (inputs.kicad_sch)
- added sheet Outputs (outputs.kicad_sch)
- added sheet Sensors (sensors.kicad_sch)
- note removed: "ADC Clamping Circuits"
- note removed: "Battery Reference"
- note removed: "Coolant Temperature Sensor"
- note removed: "Fan"
- note removed: "Fuel Injector"
- note removed: "Fuel Pump"
- note removed: "Ignition"
- note removed: "Intake Air Temp Sensor"
- note removed: "Manifold Air Pressure Sensor"
- note removed: "O2 Sensor"
- note removed: "Oxygen Sensor"
- note removed: "Safety Switches & Self-Diag"
- note removed: "Subthrottle Position Sensor"
- note removed: "Tachometer Output"
- note removed: "Throttle Position Sensor"
- note removed: "Use official speeduino, jbperf 2.1, WTMTronics DSC, etc..."
- note removed: "VR Conditioner"
- note removed: "Vehicle Speed Sensor"
- moved on the sheet: A1, C1, C2, C20, C3, C4, D1, D3, J1, JP1, U1, U2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

Commit message: Add labels
Other:
- note added: "ATTiny"
- note added: "Aux Cam Sensor (Optional)"
- note added: "ECM Connector"
- note added: "Main Processor"
- note added: "Subthrottle Driver"
- moved on the sheet: C1, C2, C3, C4, D1, D3, J1, U2, U4
