File: v4/sensors.kicad_sch (KiCad schematic)
At the start: 29 parts, among them IC1 SP721, J3 DIP8, J4 Conn_02x04_Counter_Clockwise

Commit message: V4 potential design
Parts:
- added J6, J9: Conn_01x01_Male, Connector_PinHeader_2.54mm:PinHeader_1x01_P2.54mm_Vertical, symbol Connector:Conn_01x01_Male
- added JP10, JP11, JP12, JP8, JP9: SolderJumper_2_Open, Jumper:SolderJumper-2_P1.3mm_Open_RoundedPad1.0x1.5mm, symbol Jumper:SolderJumper_2_Open
- added R3: 470, Resistor_THT:R_Axial_DIN0204_L3.6mm_D1.6mm_P5.08mm_Horizontal, symbol Device:R_Small
- added U5: 74HC4050, Package_DIP:DIP-16_W7.62mm_LongPads, symbol 4xxx:4050
Connections:
- net +5V: now also U5.1 (VCC)
- net CLUTCH-SW: now also R3.2; no longer D3.2 (A), D4.1 (K)
- net GND: now also JP12.1 (A), U5.14, U5.8 (VSS)
- net KILL-SW: now also JP8.1 (A), U5.3; no longer J3.2 (Pin_2)
- net NEUTRAL: now also JP10.1 (A), U5.7; no longer J3.5 (Pin_5)
- net SIDE-SW: now also JP9.1 (A), U5.5; no longer J3.3 (Pin_3)
- net VDOWN: now also JP11.1 (A), U5.9; no longer J3.6 (Pin_6)
- new net: J3.2 (Pin_2), JP8.2 (B), U5.2
- new net: J3.3 (Pin_3), JP9.2 (B), U5.4
- new net: J3.5 (Pin_5), JP10.2 (B), U5.6
- new net: J3.6 (Pin_6), JP11.2 (B), U5.10
- new net: J6.1 (Pin_1), JP12.2 (B), U5.11
- new net: J9.1 (Pin_1), U5.12
- new net CLUTCH-ARD-D51: D3.2 (A), D4.1 (K), R3.1
- no-connect marks 0 -> 1

Commit message: Convert to a 2 layer board
Other:
- moved on the sheet: J6, J9
Changed lines of the file:
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@@
+    (stroke (width 0) (type default) (color 0 0 0 0))
+  )
+  (wire (pts (xy 71.12 143.51) (xy 71.12 147.32))
     (stroke (width 0) (type default) (color 0 0 0 0))
   )
@@
     (stroke (width 0) (type default) (color 0 0 0 0))
   )
-  (wire (pts (xy 88.9 147.32) (xy 91.44 147.32))
+  (wire (pts (xy 88.9 147.32) (xy 91.44 143.51))
     (stroke (width 0) (type default) (color 0 0 0 0))
   )
@@
     (pin "2")
   )
-  (symbol (lib_id "Connector:Conn_01x01_Male") (at 71.12 142.24 270) (unit 1)
-    (in_bom yes) (on_board yes) (fields_autoplaced)
-    (property "Reference" "J6" (id 0) (at 72.39 142.8749 90)
-      (effects (font (size 1.27 1.27)) (justify left))
-    )
-    (property "Value" "Conn_01x01_Male" (id 1) (at 72.39 144.1449 90)
-      (effects (font (size 1.27 1.27)) (justify left) hide)
-    )
-    (property "Footprint" "Connector_PinHeader_2.54mm:PinHeader_1x01_P2.54mm_Vertical" (id 2) (at 71.12 142.24 0)
-      (effects (font (size 1.27 1.27)) hide)
-    )
-    (property "Datasheet" "~" (id 3) (at 71.12 142.24 0)
+  (symbol (lib_id "Connector:Conn_01x01_Male") (at 71.12 138.43 270) (unit 1)
+    (in_bom yes) (on_board yes) (fields_autoplaced)
+    (property "Reference" "J6" (id 0) (at 72.39 139.0649 90)
+      (effects (font (size 1.27 1.27)) (justify left))
+    )
+    (property "Value" "Conn_01x01_Male" (id 1) (at 72.39 140.3349 90)
+      (effects (font (size 1.27 1.27)) (justify left) hide)
+    )
+    (property "Footprint" "Connector_PinHeader_2.54mm:PinHeader_1x01_P2.54mm_Vertical" (id 2) (at 71.12 138.43 0)
+      (effects (font (size 1.27 1.27)) hide)
+    )
+    (property "Datasheet" "~" (id 3) (at 71.12 138.43 0)
       (effects (font (size 1.27 1.27)) hide)
     )
@@
     (pin "2")
   )
-  (symbol (lib_id "Connector:Conn_01x01_Male") (at 91.44 142.24 270) (unit 1)
-    (in_bom yes) (on_board yes) (fields_autoplaced)
-    (property "Reference" "J9" (id 0) (at 92.71 142.8749 90)
-      (effects (font (size 1.27 1.27)) (justify left))
-    )
-    (property "Value" "Conn_01x01_Male" (id 1) (at 92.71 144.1449 90)
-      (effects (font (size 1.27 1.27)) (justify left) hide)
-    )
-    (property "Footprint" "Connector_PinHeader_2.54mm:PinHeader_1x01_P2.54mm_Vertical" (id 2) (at 91.44 142.24 0)
-      (effects (font (size 1.27 1.27)) hide)
-    )
-    (property "Datasheet" "~" (id 3) (at 91.44 142.24 0)
-      (effects (font (size 1.27 1.27)) hide)
-    )
+  (symbol (lib_id "Connector:Conn_01x01_Male") (at 91.44 138.43 270) (unit 1)
+    (in_bom yes) (on_board yes) (fields_autoplaced)
+    (property "Reference" "J9" (id 0) (at 92.71 139.0649 90)
+      (effects (font (size 1.27 1.27)) (justify left))
+    )
+    (property "Value" "Conn_01x01_Male" (id 1) (at 92.71 140.3349 90)
+      (effects (font (size 1.27 1.27)) (justify left) hide)
+    )
+    (property "Footprint" "Connector_PinHeader_2.54mm:PinHeader_1x01_P2.54mm_Vertical" (id 2) (at 91.44 138.43 0)
+      (effects (font (size 1.27 1.27)) hide)
+    )
+    (property "Datasheet" "~" (id 3) (at 91.44 138.43 0)
+      (effects (font (size 1.27 1.27)) hide)
+    )
